File: Hardware/AcousticSpanner.sch (EAGLE design)
At the start: 118 parts, among them IC1 TDA7375V, IC2 TDA7375V

Commit message: Firmware updates
Other:
- note added: "FIXME: Reverse pol. on X3, X5, X11, X13"
Changed lines of the file:
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@@
 EPSRC
 ISM CDT</text>
+<text x="325.12" y="22.86" size="1.778" layer="91">FIXME: Reverse pol. on X3, X5, X11, X13</text>
 </plain>
 <instances>
